Commit message: Weekend Commit

File: src/robots/rc_car/rc_car_description/urdf/chassis/front_axle.urdf.xacro (robot description, xacro)
@@ -114,4 +114,5 @@
       <limit lower="${-degrees_45}" upper="${degrees_45}"
              effort="${steer_stall_torque}" velocity="${steer_no_load_speed}"/>
+      <!-- <dynamics damping="0.01" /> -->
     </joint>
     <transmission name="front_left_steering_trans">
@@ -156,4 +157,5 @@
       <limit lower="${-degrees_45}" upper="${degrees_45}"
              effort="${steer_stall_torque}" velocity="${steer_no_load_speed}"/>
+      <!-- <dynamics damping="0.01" /> -->
     </joint>
     <transmission name="front_right_steering_trans">

File: src/robots/rc_car/rc_car_description/urdf/chassis/rc_chassis.urdf.xacro (robot description, xacro)
@@ -36,5 +36,5 @@
   </xacro:macro>
   <!-- Used for fixing robot to Gazebo 'base_link' -->
-  <link name="world"/>
+  <!-- <link name="world"/> -->
   <!-- base_link must have geometry so that its axes can be displayed in
        rviz. -->
@@ -79,9 +79,9 @@
     <child link="chassis"/>
   </joint>
-  <joint name="world_to_chassis_joint" type="fixed">
+  <!-- <joint name="world_to_chassis_joint" type="fixed">
     <parent link="world"/>
     <child link="base_link"/>
     <origin xyz="0 0 2" />
-  </joint>
+  </joint> -->
  <xacro:include filename="$(find rc_car_description)/urdf/chassis/front_axle.urdf.xacro"/>
  <xacro:include filename="$(find rc_car_description)/urdf/chassis/rear_axle.urdf.xacro"/>

File: src/robots/rc_car/rc_car_description/urdf/chassis/rear_axle.urdf.xacro (robot description, xacro)
@@ -119,5 +119,5 @@
       <origin xyz="0 ${front_axle_W/2 - shock_y_offset} -${shock_z_offset - shock_H/2 + chassis_H/2 + ground_clearance - wheel_front_R}"/>
       <axis xyz="0 1 0"/>
-      <dynamics damping="0.01"/>
+      <dynamics damping="0.0" friction="0.0"/>
       <limit effort="${axle_eff_limit}" velocity="${axle_vel_limit}"/>
     </joint>
@@ -168,5 +168,5 @@
       <origin xyz="0 -${front_axle_W/2 - shock_y_offset} -${shock_z_offset - shock_H/2 + chassis_H/2 + ground_clearance - wheel_front_R}"/>
       <axis xyz="0 1 0"/>
-      <dynamics damping="0.01"/>
+      <dynamics damping="0.0" friction="0.0"/>
       <limit effort="${axle_eff_limit}" velocity="${axle_vel_limit}"/>
     </joint>
